File: AGB-64M_SUB_BOARD.kicad_pcb (KiCad board)
At the start: 2 copper layers, 45.5 x 27.8 mm, 9 parts, among them J1 AXK640347YG, U1 256KFRAM FM18W08, U2 AGB512K FLASH U2

Commit message: Fix back silkscreen type (サブカートリッヅS changed to サブカートリッジS)
Other:
- board text added: "サブカートリッジS"
- board text removed: "サブカートリッヅS"
Changed lines of the file:
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@@
     (effects (font (size 1.45 1.6) (thickness 0.2) bold) (justify left bottom mirror))
   )
-  (gr_text "サブカートリッヅS" (at 67.93 77) (layer "B.SilkS")
+  (gr_text "サブカートリッジS" (at 67.93 77) (layer "B.SilkS")
     (effects (font (size 1.45 1.6) (thickness 0.25) bold) (justify left bottom mirror))
   )
